File: STLink-Edge/STLink-Edge.kicad_sch (KiCad schematic)
At the start: 2 parts, among them J1 Conn_edge_socket, J2 Conn_STLink

Commit message: edgelink 2.1
Parts:
- removed J2: Conn_STLink, Connector_PinHeader_2.54mm:PinHeader_1x04_P2.54mm_Vertical, symbol Connector:Conn_01x04_Socket
- added J3: Conn_STLink2, Connector_PinHeader_2.54mm:PinHeader_1x05_P2.54mm_Vertical, symbol Connector:Conn_01x05_Socket
- added SW1: SW_Push_SPDT, Connector_PinHeader_2.54mm:PinHeader_1x03_P2.54mm_Vertical, symbol Switch:SW_Push_SPDT
Connections:
- net +3.3V: now also J3.2 (Pin_2), SW1.3 (C); no longer J1.1 (Pin_1), J1.3 (Pin_3), J1.6 (Pin_6), J1.8 (Pin_8)
- net GND: now also J3.3 (Pin_3)
- net SWCLK: now also J3.5 (Pin_5)
- net SWDIO: now also J3.4 (Pin_4)
- new net +5V: J3.1 (Pin_1), SW1.1 (A)
- new net Boot: J1.1 (Pin_1), J1.3 (Pin_3), J1.6 (Pin_6), J1.8 (Pin_8), SW1.2 (B)
