File: STM32-iButton/STM32-iButton.kicad_sch (KiCad schematic)
At the start: 10 parts, among them J1 Conn_SWD, J2 Conn_SWD, P1 USB_C_2.0, SW1 Button_user, U1 STM32L052C8Tx, U2 AMS1117-3.3

Commit message: updated
Parts:
- added SW2, SW3: Button_user, Button_Switch_SMD:SW_SPST_SKQG_WithoutStem, symbol Switch:SW_Push_Dual
- J1, J2: footprint (none) -> wyw-conn:SWD5-Gold
- P1: footprint (none) -> Connector_USB:USB_C_Plug_JAE_DX07P024AJ1
- R1: value 10k -> 1.5k
- SW1: footprint (none) -> Button_Switch_SMD:SW_SPST_SKQG_WithoutStem
- U2: footprint Package_TO_SOT_SMD:SOT-223-3_TabPin2 -> Package_TO_SOT_SMD:SOT-89-3_Handsoldering
Connections:
- net +3.3V: now also R1.1
- net D+: now also R1.2, U1.33 (PA12)
- net D-: now also U1.32 (PA11)
- net SWCLK: now also U1.37 (PA14)
- net SWDIO: now also U1.34 (PA13)
- net CC: no longer names the net of P1.A5 (CC)
- net VCONN: no longer names the net of P1.B5 (VCONN)
- no-connect marks 1 -> 3
Other:
- moved on the sheet: SW1, U1

Commit message: updated
Parts:
- C1, C2: footprint (none) -> Capacitor_SMD:C_0603_1608Metric_Pad1.08x0.95mm_HandSolder
- P1: footprint Connector_USB:USB_C_Plug_JAE_DX07P024AJ1 -> wyw-conn:USB_C_Male
- R1, R2: footprint (none) -> Resistor_SMD:R_0603_1608Metric_Pad0.98x0.95mm_HandSolder
Connections:
- net GND: now also SW1.2, SW1.4, SW2.2, SW2.4, SW3.2, SW3.4
- net Btn2: now reaches SW2.1
- net Btn2: now also SW2.3, U1.3 (PC14)
- net Btn1: now reaches SW1.1
- net Btn1: now also SW1.3, U1.2 (PC13)
- net Btn3: now reaches SW3.1
- net Btn3: now also SW3.3, U1.4 (PC15)
- no-connect marks 3 -> 34
Other:
- moved on the sheet: SW1, SW2, SW3

Commit message: critical fix: 5V power
Connections:
- net +3.3V: no longer J1.1 (Pin_1), J2.1 (Pin_1)
- net +5V: now reaches C2.1, P1.A4 (VBUS), P1.A9 (VBUS), P1.B4 (VBUS), P1.B9 (VBUS), U2.3 (VI)
- net +5V: now also J1.1 (Pin_1), J2.1 (Pin_1)
Changed lines of the file:
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@@
+	)
+	(junction
+		(at 238.76 66.04)
+		(diameter 0)
+		(color 0 0 0 0)
 	)
 	(junction
@@
 	(wire
 		(pts
-			(xy 228.6 66.04) (xy 241.3 66.04)
+			(xy 228.6 66.04) (xy 238.76 66.04)
 		)
 		(stroke
@@
 	(wire
 		(pts
+			(xy 238.76 66.04) (xy 241.3 66.04)
+		)
+		(stroke
+			(width 0)
+			(type default)
+		)
+	)
+	(wire
+		(pts
 			(xy 163.83 105.41) (xy 163.83 107.95)
 		)
@@
 		(pts
 			(xy 209.55 73.66) (xy 209.55 76.2)
+		)
+		(stroke
+			(width 0)
+			(type default)
+		)
+	)
+	(wire
+		(pts
+			(xy 238.76 63.5) (xy 238.76 66.04)
 		)
 		(stroke
@@
 			)
 			(justify right)
+		)
+	)
+	(symbol
+		(lib_id "power:+3.3V")
+		(at 232.41 29.21 0)
+		(unit 1)
+		(exclude_from_sim no)
+		(in_bom yes)
+		(on_board yes)
+		(dnp no)
+		(fields_autoplaced yes)
+		(property "Reference" "#PWR014"
+			(at 232.41 33.02 0)
+			(effects
+				(font
+					(size 1.27 1.27)
+				)
+				(hide yes)
+			)
+		)
+		(property "Value" "+5V"
+			(at 232.41 25.0769 0)
+			(effects
+				(font
+					(size 1.27 1.27)
+				)
+			)
+		)
+		(property "Footprint" ""
+			(at 232.41 29.21 0)
+			(effects
+				(font
+					(size 1.27 1.27)
+				)
+				(hide yes)
+			)
+		)
+		(property "Datasheet" ""
+			(at 232.41 29.21 0)
+			(effects
+				(font
+					(size 1.27 1.27)
+				)
+				(hide yes)
+			)
+		)
+		(property "Description" "Power symbol creates a global label with name \"+3.3V\""
+			(at 232.41 29.21 0)
+			(effects
+				(font
+					(size 1.27 1.27)
+				)
+				(hide yes)
+			)
+		)
+		(pin "1"
+		)
+		(instances
+			(project "STM32-iButton"
+				(path "/4efb9682-f06b-455d-b5a5-d5184deb6e4d"
+					(reference "#PWR014")
+					(unit 1)
+				)
+			)
 		)
 	)
@@
 	(symbol
 		(lib_id "power:+3.3V")
-		(at 232.41 29.21 0)
+		(at 255.27 29.21 0)
 		(unit 1)
 		(exclude_from_sim no)
@@
 		(dnp no)
 		(fields_autoplaced yes)
-		(property "Reference" "#PWR04"
-			(at 232.41 33.02 0)
-			(effects
-				(font
-					(size 1.27 1.27)
-				)
-				(hide yes)
-			)
-		)
-		(property "Value" "+3.3V"
-			(at 232.41 25.0769 0)
+		(property "Reference" "#PWR015"
+			(at 255.27 33.02 0)
+			(effects
+				(font
+					(size 1.27 1.27)
+				)
+				(hide yes)
+			)
+		)
+		(property "Value" "+5V"
+			(at 255.27 25.0769 0)
 			(effects
 				(font
@@
 		)
 		(property "Footprint" ""
-			(at 232.41 29.21 0)
+			(at 255.27 29.21 0)
 			(effects
 				(font
@@
 		)
 		(property "Datasheet" ""
-			(at 232.41 29.21 0)
+			(at 255.27 29.21 0)
 			(effects
 				(font
@@
 		)
 		(property "Description" "Power symbol creates a global label with name \"+3.3V\""
-			(at 232.41 29.21 0)
+			(at 255.27 29.21 0)
 			(effects
 				(font
@@
 			(project "STM32-iButton"
 				(path "/4efb9682-f06b-455d-b5a5-d5184deb6e4d"
-					(reference "#PWR04")
+					(reference "#PWR015")
 					(unit 1)
 				)
@@
 				(path "/4efb9682-f06b-455d-b5a5-d5184deb6e4d"
 					(reference "R1")
+					(unit 1)
+				)
+			)
+		)
+	)
+	(symbol
+		(lib_id "power:+3.3V")
+		(at 238.76 63.5 0)
+		(unit 1)
+		(exclude_from_sim no)
+		(in_bom yes)
+		(on_board yes)
+		(dnp no)
+		(fields_autoplaced yes)
+		(property "Reference" "#PWR013"
+			(at 238.76 67.31 0)
+			(effects
+				(font
+					(size 1.27 1.27)
+				)
+				(hide yes)
+			)
+		)
+		(property "Value" "+5V"
+			(at 238.76 59.3669 0)
+			(effects
+				(font
+					(size 1.27 1.27)
+				)
+			)
+		)
+		(property "Footprint" ""
+			(at 238.76 63.5 0)
+			(effects
+				(font
+					(size 1.27 1.27)
+				)
+				(hide yes)
+			)
+		)
+		(property "Datasheet" ""
+			(at 238.76 63.5 0)
+			(effects
+				(font
+					(size 1.27 1.27)
+				)
+				(hide yes)
+			)
+		)
+		(property "Description" "Power symbol creates a global label with name \"+3.3V\""
+			(at 238.76 63.5 0)
+			(effects
+				(font
+					(size 1.27 1.27)
+				)
+				(hide yes)
+			)
+		)
+		(pin "1"
+		)
+		(instances
+			(project "STM32-iButton"
+				(path "/4efb9682-f06b-455d-b5a5-d5184deb6e4d"
+					(reference "#PWR013")
 					(unit 1)
 				)
@@
 					(unit 1)
 				)
-			)
-		)
-	)
-	(symbol
-		(lib_id "power:+3.3V")
-		(at 255.27 29.21 0)
-		(unit 1)
-		(exclude_from_sim no)
-		(in_bom yes)
-		(on_board yes)
-		(dnp no)
-		(fields_autoplaced yes)
-		(property "Reference" "#PWR05"
-			(at 255.27 33.02 0)
-			(effects
-				(font
-					(size 1.27 1.27)
-				)
-				(hide yes)
-			)
-		)
-		(property "Value" "+3.3V"
-			(at 255.27 25.0769 0)
-			(effects
-				(font
-					(size 1.27 1.27)
-				)
-			)
-		)
-		(property "Footprint" ""
-			(at 255.27 29.21 0)
-			(effects
-				(font
-					(size 1.27 1.27)
-				)
-				(hide yes)
-			)
-		)
-		(property "Datasheet" ""
-			(at 255.27 29.21 0)
-			(effects
-				(font
-					(size 1.27 1.27)
-				)
-				(hide yes)
-			)
-		)
-		(property "Description" "Power symbol creates a global label with name \"+3.3V\""
-			(at 255.27 29.21 0)
-			(effects
-				(font
-					(size 1.27 1.27)
-				)
-				(hide yes)
-			)
-		)
-		(pin "1"
-		)
-		(instances
-			(project "STM32-iButton"
-				(path "/4efb9682-f06b-455d-b5a5-d5184deb6e4d"
-					(reference "#PWR05")
-					(unit 1)
-				)

Commit message: updated
Parts:
- added C3, C4, C5: 4.7uF, Capacitor_SMD:C_0603_1608Metric_Pad1.08x0.95mm_HandSolder, symbol Device:C_Small
Connections:
- net Btn1: now also C3.1
- net Btn2: now also C4.1
- net Btn3: now also C5.1
- net GND: now also C3.2, C4.2, C5.2
