File: STM32-iButton/STM32-iButton.kicad_pcb (KiCad board)
At the start: 2 copper layers, 49.7 x 18 mm, 12 parts, among them J1 Conn_SWD, J2 Conn_SWD, P1 USB_C_2.0, SW1 Button_user, SW2 Button_user, SW3 Button_user, U1 STM32L052C8Tx, U2 AMS1117-3.3

Commit message: updated
Parts:
- added C3: 4.7uF, Capacitor_SMD:C_0603_1608Metric_Pad1.08x0.95mm_HandSolder, F.Cu at (71.8, 43.5)
- added C4: 4.7uF, Capacitor_SMD:C_0603_1608Metric_Pad1.08x0.95mm_HandSolder, F.Cu at (83.0, 43.5)
- added C5: 4.7uF, Capacitor_SMD:C_0603_1608Metric_Pad1.08x0.95mm_HandSolder, F.Cu at (87.5, 43.5)
Routing:
- net /Btn1: track 12.0 -> 14.9 mm
- net /Btn2: track 25.0 -> 27.2 mm
- net /Btn3: track 36.5 -> 38.4 mm
- net GND: vias 34 -> 38

Commit message: updated silks
Other:
- board text added: "iButton v2.2 2024.04 by Leo"
- board text removed: "iButton v2.1 2024.03 by Leo"
Changed lines of the file:
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@@
 		)
 	)
-	(gr_text "iButton v2.1\n2024.03\nby Leo"
+	(gr_text "iButton v2.2\n2024.04\nby Leo"
 		(at 62.5 40 0)
 		(layer "F.SilkS")
