File: STM32-iButton/STM32-iButton-FrontVer.kicad_pcb (KiCad board)
At the start: 2 copper layers, 49.7 x 18 mm, 15 parts, among them J1 Conn_SWD, J2 Conn_SWD, P1 USB_C_2.0, SW1 Button_user, SW2 Button_user, SW3 Button_user, U1 STM32L052C8Tx, U2 AMS1117-3.3

Commit message: add front ver
Parts:
- U1: moved to F.Cu
- moved U1 0.75 mm to (62.8, 39.0)
Routing:
- net GND: track 38.3 -> 111.9 mm, vias 38 -> 45
- net /Boot: track 49.1 -> 58.3 mm, vias 3 -> 4
- net /SWCLK: track 43.8 -> 52.9 mm, vias 1 -> 2
- net /Btn1: track 14.9 -> 20.7 mm, vias 1 -> 2
- net /SWDIO: track 52.6 -> 57.0 mm, vias 1 -> 2
- net /Btn2: track 27.2 -> 31.4 mm, vias 1 -> 0
- net /Btn3: track 38.4 -> 42.1 mm, vias 1 -> 2
- net /D+: track 23.6 -> 25.3 mm, vias 1 -> 0
- net /D-: track 23.2 -> 24.2 mm, vias 1 -> 0
- net +3.3V: track 40.4 -> 39.7 mm, vias 3 -> 2
Other:
- board text added: "iButton v2.3 2024.04 by Leo"
- board text removed: "iButton v2.2 2024.04 by Leo"
