File: EdgeLink2/STLink-Edge.kicad_pcb (KiCad board)
At the start: 2 copper layers, 30 x 15 mm, 3 parts, among them J1 Conn_edge_socket, J3 Conn_STLink2, SW1 SW_Push_SPDT

Commit message: updated
Other:
- board text added: "EdgeLink v2.1 for STLink-V2 2024.04 by Leo"
- board text removed: "STLink-V2 EdgeDebugger 2024.03 v2.1 by Leo"
Changed lines of the file:
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@@
 		(layer "Margin")
 	)
-	(gr_text "STLink-V2\nEdgeDebugger\n2024.03\nv2.1 by Leo"
-		(at 63 57 0)
+	(gr_text "EdgeLink v2.1\nfor STLink-V2\n2024.04 by Leo"
+		(at 63 56.5 0)
 		(layer "B.SilkS")
 		(effects

Commit message: updated
Other:
- board size 30 x 15 mm -> 37 x 15 mm
Changed lines of the file:
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@@
 	)
 	(gr_arc
-		(start 43 62)
-		(mid 41.585786 61.414214)
-		(end 41 60)
+		(start 36 62)
+		(mid 34.585786 61.414214)
+		(end 34 60)
 		(stroke
 			(width 0.05)
@@
 	)
 	(gr_arc
-		(start 41 49)
-		(mid 41.585786 47.585786)
-		(end 43 47)
+		(start 34 49)
+		(mid 34.585786 47.585786)
+		(end 36 47)
 		(stroke
 			(width 0.05)
@@
 	)
 	(gr_line
-		(start 41 60)
-		(end 41 49)
+		(start 34 60)
+		(end 34 49)
 		(stroke
 			(width 0.05)
@@
 	)
 	(gr_arc
-		(start 41.5 49)
-		(mid 41.93934 47.93934)
-		(end 43 47.5)
+		(start 34.5 49)
+		(mid 34.93934 47.93934)
+		(end 36 47.5)
 		(stroke
 			(width 0.1)
@@
 	)
 	(gr_line
-		(start 41.5 60)
-		(end 41.5 49)
+		(start 34.5 60)
+		(end 34.5 49)
 		(stroke
 			(width 0.1)
@@
 	)
 	(gr_arc
-		(start 43 61.5)
-		(mid 41.93934 61.06066)
-		(end 41.5 60)
+		(start 36 61.5)
+		(mid 34.93934 61.06066)
+		(end 34.5 60)
 		(stroke
 			(width 0.1)
